Commit message: 含slam建图功能

File: ros2_projects/project_1/src/my_robot_description/urdf/robot.urdf.xacro (robot description, xacro)
@@ -4,4 +4,5 @@
   <xacro:include filename="$(find my_robot_description)/urdf/wheels.xacro"/>
   <xacro:include filename="$(find my_robot_description)/urdf/sensors.xacro"/>
+  <xacro:include filename="$(find my_robot_description)/urdf/gazebo.xacro"/>
   <xacro:property name="body_length" value="0.50"/>
   <xacro:property name="body_width" value="0.34"/>
@@ -11,11 +12,24 @@
   <xacro:property name="wheel_width" value="0.04"/>
   <xacro:property name="wheel_mass" value="0.6"/>
-  <xacro:property name="wheel_x" value="0.0"/>
+  <xacro:property name="wheel_x" value="0.04"/>
   <xacro:property name="wheel_y_offset" value="${body_width / 2.0 + wheel_width / 2.0}"/>
   <xacro:property name="wheel_z" value="${-body_height / 2.0}"/>
-  <xacro:property name="caster_x" value="${-body_length / 2.5}"/>
+  <xacro:property name="rear_caster_x" value="${-body_length / 2.3}"/>
+  <xacro:property name="front_caster_x" value="${body_length / 2.6}"/>
   <xacro:property name="caster_z" value="${-(body_height / 2.0 + 0.04)}"/>
   <xacro:property name="lidar_height" value="${body_height / 2.0 + 0.08}"/>
   <xacro:property name="camera_height" value="${body_height / 2.0 + 0.14}"/>
+  <xacro:property name="lidar_min_angle" value="-3.14159"/>
+  <xacro:property name="lidar_max_angle" value="3.14159"/>
+  <xacro:property name="lidar_samples" value="720"/>
+  <xacro:property name="lidar_range_min" value="0.05"/>
+  <xacro:property name="lidar_range_max" value="8.0"/>
+  <xacro:property name="lidar_update_rate" value="10.0"/>
+  <xacro:property name="camera_width" value="640"/>
+  <xacro:property name="camera_height_px" value="480"/>
+  <xacro:property name="camera_hfov" value="1.047"/>
+  <xacro:property name="camera_near_clip" value="0.05"/>
+  <xacro:property name="camera_far_clip" value="20.0"/>
+  <xacro:property name="camera_update_rate" value="15.0"/>
   <xacro:chassis
     length="${body_length}"
@@ -40,5 +54,13 @@
     mass="${wheel_mass}"/>
   <xacro:caster_wheel
-    x="${caster_x}"
+    prefix="rear"
+    x="${rear_caster_x}"
+    y="0.0"
+    z="${caster_z}"
+    radius="0.04"
+    mass="0.2"/>
+  <xacro:caster_wheel
+    prefix="front"
+    x="${front_caster_x}"
     y="0.0"
     z="${caster_z}"
@@ -49,3 +71,26 @@
     lidar_height="${lidar_height}"
     camera_height="${camera_height}"/>
+  <xacro:gazebo_diff_drive
+    wheel_separation="${2.0 * wheel_y_offset}"
+    wheel_radius="${wheel_radius}"/>
+  <xacro:gazebo_joint_state_publisher/>
+  <xacro:gazebo_lidar
+    topic_name="/scan"
+    update_rate="${lidar_update_rate}"
+    min_angle="${lidar_min_angle}"
+    max_angle="${lidar_max_angle}"
+    samples="${lidar_samples}"
+    range_min="${lidar_range_min}"
+    range_max="${lidar_range_max}"
+    visualize="true"/>
+  <xacro:gazebo_camera
+    image_topic="/camera/image_raw"
+    camera_info_topic="/camera/camera_info"
+    update_rate="${camera_update_rate}"
+    width="${camera_width}"
+    height="${camera_height_px}"
+    hfov="${camera_hfov}"
+    near_clip="${camera_near_clip}"
+    far_clip="${camera_far_clip}"
+    visualize="true"/>
 </robot>

File: ros2_projects/project_1/src/my_robot_description/urdf/sensors.xacro (robot description, xacro)
@@ -56,4 +56,10 @@
       <origin xyz="${body_length / 2.5} 0 ${camera_height}" rpy="0 0 0"/>
     </joint>
+    <link name="camera_optical_link"/>
+    <joint name="camera_optical_joint" type="fixed">
+      <parent link="camera_link"/>
+      <child link="camera_optical_link"/>
+      <origin xyz="0 0 0" rpy="-1.5708 0 -1.5708"/>
+    </joint>
   </xacro:macro>
 </robot>

File: ros2_projects/project_1/src/my_robot_description/urdf/wheels.xacro (robot description, xacro)
@@ -37,6 +37,6 @@
     </joint>
   </xacro:macro>
-  <xacro:macro name="caster_wheel" params="x y z radius mass">
-    <link name="caster_link">
+  <xacro:macro name="caster_wheel" params="prefix x y z radius mass">
+    <link name="${prefix}_caster_link">
       <visual>
         <origin xyz="0 0 0" rpy="0 0 0"/>
@@ -66,7 +66,7 @@
       </inertial>
     </link>
-    <joint name="caster_joint" type="fixed">
+    <joint name="${prefix}_caster_joint" type="fixed">
       <parent link="base_link"/>
-      <child link="caster_link"/>
+      <child link="${prefix}_caster_link"/>
       <origin xyz="${x} ${y} ${z}" rpy="0 0 0"/>
     </joint>
